File: Hardware/CAN.kicad_sch (KiCad schematic)
At the start: 0 parts

Commit message: Finished the ISOW1044 Schematic
- Ported over Kostadin's schematic

Co-authored-by: Kostadin Madjovski <155325994+bivein@users.noreply.github.com>
Parts:
- added C16 (x2), C25, C29: 100n, symbol Device:C
- added C17: 4.7n, symbol Device:C
- added C17: 10u, symbol Device:C
- added C22, C28: 1u, symbol Device:C
- added C23, C24: 10n, symbol Device:C
- added D2: D_TVS_Dual_AAC, symbol Device:D_TVS_Dual_AAC
- added FB1, FB2, FB3, FB4: FerriteBead, BLM15EX331SN1D:BEADC1005X55N, symbol Device:FerriteBead
- added R10, R9: 60, symbol Device:R
- added R11: 5k, symbol Device:R
- added U4: ISOW1044, Package_SO:SOIC-20W_7.5x12.8mm_P1.27mm, symbol Interface_CAN_LIN:ISOW1044
Connections:
- new net: C16.1, C24.1, C28.1, FB3.1, U4.12 (VISOOUT), U4.13 (VSIN)
- new net: C16.2, C24.2, C28.2, FB4.2, U4.11 (GND2)
- new net: C16.1, FB2.2, R11.1, U4.1 (VIO)
- new net: R11.2, U4.8 (EN/FLT)
- new net: C17.1, C22.1, C23.1, FB1.1
- new net: C25.1, C29.1, FB3.2, U4.20 (VISOIN)
- new net: C17.1, R10.1, R9.2
- new net +3V3: FB2.1
- new net +5V: FB1.2, U4.9 (VDD)
- new net CAN1_RX: U4.5 (RXD)
- new net CAN1_TX: U4.3 (TXD)
- new net CANGND: C17.2, C25.2, C29.2, D2.3 (common), FB4.1, U4.15 (GISOIN), U4.16 (GISOIN), U4.17 (GISOIN)
- new net CANH_+: D2.2 (A2), R9.1, U4.19 (CANH)
- new net CANL_-: D2.1 (A1), R10.2, U4.18 (CANL)
- new net CAN_IN: U4.2 (IN)
- new net CAN_STB: U4.4 (STB)
- new net GND: C16.2, C17.2, C22.2, C23.2, U4.10 (GND1), U4.6 (GNDIO)
- no-connect marks 0 -> 1
Other:
- note added: "- CANH/L_+/- are a differential pair (120 ohm differential, 60 ohm odd-mode), and as such trace width, spacing etc will need to be calculated at route-time - The abundance of ferrites is puzzling, but is what's recommended in the datasheet. The ferrites will all be 0603 package, but the exact bead will have to be determined by the 100MHz impedance, and ZRX curve. - The ISOW1044 Datasheet recommen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"
- note added: "Design Notes"
- note added: "Global/Hierarchical Labels"
- note added: "Isolated CAN Transciever"
- note added: "Isolation Barrier"

Commit message: Finished final touches on schematic.
- Schematic is complete (NOT yet checked by Yassa/Val)
- ERC check is complete, understandable errors excused w/ comments
- Final schematic formatting complete

Co-authored-by: Kostadin Madjovski <155325994+bivein@users.noreply.github.com>
Parts:
- removed C16: 100n, symbol Device:C
- removed C17: 10u, symbol Device:C
- added C26: 100n, symbol Device:C
- added C27: 10u, symbol Device:C
- renumbered D2 to TVS2
Connections:
- net GND: now also C26.2, C27.2
- net at FB2.2, R11.1, U4.1 (VIO): now also C26.1
- net at C22.1, C23.1, FB1.1: now also U4.9 (VDD), C27.1
- net +3V3 renamed 3v3
- net +5V renamed 5v0
- net 5v0: no longer U4.9 (VDD)
Other:
- company: (none) -> NJIT Solar Car
- title: (none) -> CAN IO Board | CAN Transciever
- moved on the sheet: FB1
