File: Hardware/Connectors.kicad_sch (KiCad schematic)
At the start: 0 parts

Commit message: Finished final touches on schematic.
- Schematic is complete (NOT yet checked by Yassa/Val)
- ERC check is complete, understandable errors excused w/ comments
- Final schematic formatting complete

Co-authored-by: Kostadin Madjovski <155325994+bivein@users.noreply.github.com>
Parts:
- added C20, C21: 1u, symbol Device:C_Small_US
- added DIP1: SW_DIP_x03, symbol Switch:SW_DIP_x03
- added FILTER1: ECMF2-40A100N6, symbol symbols:ECMF2-40A100N6
- added J3: Conn_01x05, symbol Connector_Generic:Conn_01x05
- added J4: TC2030, Connector:Tag-Connect_TC2030-IDC-NL_2x03_P1.27mm_Vertical, symbol Connector:TC2030
- added J5: Conn_01x03, symbol Connector_Generic:Conn_01x03
- added J6: USB_C_Receptacle_USB2.0_14P, symbol Connector:USB_C_Receptacle_USB2.0_14P
- added R13, R14: 5.1k, symbol Device:R_Small_US
- added R15, R17: 10k, symbol Device:R_Small_US
- added R16: 20k, symbol Device:R_Small_US
- added SW6, SW7: SW_Push, symbol Switch:SW_Push
- added TD1: Conn_01x02, symbol Connector_Generic:Conn_01x02
- added TVS3, TVS4, TVS5: ESDS314DBVR, symbol symbols:ESDS314DBVR
- added WAGO1, WAGO2: 2606, symbol Connector_Generic:Conn_01x02
- added WAGO3, WAGO4, WAGO5: 2601, symbol Connector_Generic:Conn_01x02
Connections:
- new net: R15.2, SW6.1
- new net: J6.A5 (CC1), R13.2
- new net: J6.A4 (VBUS), J6.A9 (VBUS), J6.B4 (VBUS), J6.B9 (VBUS)
- new net: J6.B5 (CC2), R14.2
- new net: R17.2, SW7.2
- new net 3v3: DIP1.4, DIP1.5, DIP1.6, J4.1
- new net 5v0: C20.1, SW6.2
- new net CANH_+: TD1.1 (Pin_1)
- new net CANL_-: TD1.2 (Pin_2)
- new net CAN_ADDR0: DIP1.3
- new net CAN_ADDR1: DIP1.2
- new net CAN_ADDR2: DIP1.1
- new net GND: C21.2, FILTER1.3 (GND), FILTER1.4 (GND), J4.3, J4.5, J6.A1 (GND), J6.A12 (GND), J6.B1 (GND), J6.B12 (GND), J6.S1 (SHIELD), R13.1, R14.1, R16.2, SW7.1, TVS3.2 (GND), TVS4.2 (GND), TVS5.2 (GND), WAGO1.2 (Pin_2), WAGO2.2 (Pin_2), WAGO3.2 (Pin_2), WAGO4.2 (Pin_2), WAGO5.2 (Pin_2)
- new net GPIO0: J3.1 (Pin_1), TVS4.5 (IN4)
- new net GPIO1: J3.2 (Pin_2), TVS4.4 (IN3)
- new net GPIO2: J3.3 (Pin_3), TVS4.3 (IN2)
- new net GPIO3: J3.4 (Pin_4), TVS4.1 (IN1)
- new net GPIO4: J3.5 (Pin_5), TVS3.5 (IN4)
- new net HighDriveOut1: WAGO1.1 (Pin_1)
- new net HighDriveOut2: WAGO2.1 (Pin_1)
- new net LowDrive1: WAGO3.1 (Pin_1)
- new net LowDrive2: WAGO4.1 (Pin_1)
- new net LowDrive3: WAGO5.1 (Pin_1)
- new net NRST: C21.1, J4.6, J5.3 (Pin_3), R17.1, TVS5.3 (IN2)
- new net SWCLK: J4.4, J5.2 (Pin_2), TVS5.4 (IN3)
- new net SWDIO: J4.2, J5.1 (Pin_1), TVS5.5 (IN4)
- new net USBD+: FILTER1.2 (DN_C), J6.A6 (D+), J6.B6 (D+)
- new net USBD-: FILTER1.1 (DP_C), J6.A7 (D-), J6.B7 (D-)
- new net USB_DM-: FILTER1.6 (DP_IC)
- new net USB_DP+: FILTER1.5 (DN_IC)
- new net WKUP: C20.2, R15.1, R16.1
- no-connect marks 0 -> 5
Other:
- note added: "- The CANH and CANL lines are connected to the 2 pin TD connector. As of date the pinout is TBD, might be swapped. - The CAN Address Dip Switch should control the least significant 3 bits of the board's CAN ID. This will allow upto 8 CAN ID variations, as per the reqs. - The GPIOs are exposed, and thus have a 4 channel unidirectional TVS diode array. PWR voltage is 3.6V. - Since the SWD pins are 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"
- note added: "CAN Address Dip Switch"
- note added: "CAN Lines (TD connector)"
- note added: "Design Notes"
- note added: "GPIO Connector (TBD)"
- note added: "Global/Hierarchical Labels"
- note added: "High Current Outputs"
- note added: "Low Current Outputs"
- note added: "SWD"
- note added: "WKUP and RST"
- company: (none) -> NJIT Solar Car
- title: (none) -> CAN IO Board | Connectors
