File: CANIO-Board/CAN.kicad_sch (KiCad schematic)
At the start: 14 parts, among them U5 NME1

Commit message: Did some of the layout
Co-authored-by: Kostadin Madjovski <155325994+bivein@users.noreply.github.com>
Parts:
- C13: footprint Capacitor_SMD:C_0603_1608Metric_Pad1.08x0.95mm_HandSolder -> Capacitor_SMD:CP_Elec_4x4.5
- FILTER1: footprint footprints:SOIC127P600X175-16N -> footprints:ECMF02-2AMX6_QFN-6L
- U2: renamed from U5; footprint nme1footprint:NME1S -> footprints:NME1S
Connections:
- net CANH_+: now also TVS1.2 (A2)
- net CANL_-: now also TVS1.1 (A1)
- net FILTERED_CAN+: no longer TVS1.2 (A2)
- net FILTERED_CAN-: no longer TVS1.1 (A1)
Other:
- moved on the sheet: FILTER1, TVS1
Changed lines of the file:
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@@
+	)
+	(junction
+		(at 162.56 95.25)
+		(diameter 0)
+		(color 0 0 0 0)
+	)
+	(junction
+		(at 196.85 78.74)
+		(diameter 0)
+		(color 0 0 0 0)
 	)
 	(junction
@@
 	)
 	(junction
-		(at 170.18 95.25)
-		(diameter 0)
-		(color 0 0 0 0)
-	)
-	(junction
 		(at 128.27 45.72)
-		(diameter 0)
-		(color 0 0 0 0)
-	)
-	(junction
-		(at 185.42 95.25)
 		(diameter 0)
 		(color 0 0 0 0)
@@
 	)
 	(junction
-		(at 160.02 78.74)
+		(at 214.63 76.2)
 		(diameter 0)
 		(color 0 0 0 0)
 	)
 	(junction
-		(at 180.34 76.2)
+		(at 193.04 95.25)
 		(diameter 0)
 		(color 0 0 0 0)
@@
 	(wire
 		(pts
+			(xy 162.56 95.25) (xy 193.04 95.25)
+		)
+		(stroke
+			(width 0)
+			(type default)
+		)
+	)
+	(wire
+		(pts
 			(xy 173.99 59.69) (xy 173.99 62.23)
 		)
@@
 	(wire
 		(pts
-			(xy 213.36 76.2) (xy 226.06 76.2)
+			(xy 190.5 76.2) (xy 214.63 76.2)
 		)
 		(stroke
@@
 		)
 	)
-	(wire
-		(pts
-			(xy 185.42 95.25) (xy 170.18 95.25)
-		)
-		(stroke
-			(width 0)
-			(type default)
-		)
-	)
 	(bus
 		(pts
@@
 	(wire
 		(pts
-			(xy 170.18 92.71) (xy 170.18 95.25)
-		)
-		(stroke
-			(width 0)
-			(type default)
-		)
-	)
-	(wire
-		(pts
 			(xy 185.42 55.88) (xy 185.42 62.23)
 		)
@@
 	(wire
 		(pts
-			(xy 160.02 78.74) (xy 160.02 88.9)
-		)
-		(stroke
-			(width 0)
-			(type default)
-		)
-	)
-	(wire
-		(pts
 			(xy 185.42 45.72) (xy 191.77 45.72)
 		)
@@
 	(wire
 		(pts
-			(xy 161.29 88.9) (xy 160.02 88.9)
-		)
-		(stroke
-			(width 0)
-			(type default)
-		)
-	)
-	(wire
-		(pts
 			(xy 113.03 81.28) (xy 115.57 81.28)
 		)
@@
 	(wire
 		(pts
+			(xy 214.63 76.2) (xy 226.06 76.2)
+		)
+		(stroke
+			(width 0)
+			(type default)
+		)
+	)
+	(wire
+		(pts
+			(xy 196.85 78.74) (xy 196.85 87.63)
+		)
+		(stroke
+			(width 0)
+			(type default)
+		)
+	)
+	(wire
+		(pts
 			(xy 119.38 62.23) (xy 119.38 57.15)
 		)
@@
 	(wire
 		(pts
-			(xy 160.02 78.74) (xy 187.96 78.74)
+			(xy 144.78 78.74) (xy 165.1 78.74)
 		)
 		(stroke
@@
 	(wire
 		(pts
-			(xy 185.42 95.25) (xy 215.9 95.25)
-		)
-		(stroke
-			(width 0)
-			(type default)
-		)
-	)
-	(wire
-		(pts
 			(xy 124.46 54.61) (xy 128.27 54.61)
 		)
@@
 	(wire
 		(pts
-			(xy 170.18 95.25) (xy 148.59 95.25)
-		)
-		(stroke
-			(width 0)
-			(type default)
-		)
-	)
-	(wire
-		(pts
-			(xy 215.9 81.28) (xy 215.9 95.25)
+			(xy 148.59 95.25) (xy 162.56 95.25)
+		)
+		(stroke
+			(width 0)
+			(type default)
+		)
+	)
+	(wire
+		(pts
+			(xy 193.04 81.28) (xy 193.04 95.25)
 		)
 		(stroke
@@
 	(wire
 		(pts
+			(xy 205.74 91.44) (xy 205.74 95.25)
+		)
+		(stroke
+			(width 0)
+			(type default)
+		)
+	)
+	(wire
+		(pts
 			(xy 128.27 62.23) (xy 119.38 62.23)
 		)
@@
 	(wire
 		(pts
-			(xy 179.07 88.9) (xy 180.34 88.9)
-		)
-		(stroke
-			(width 0)
-			(type default)
-		)
-	)
-	(wire
-		(pts
-			(xy 213.36 78.74) (xy 226.06 78.74)
+			(xy 190.5 78.74) (xy 196.85 78.74)
 		)
 		(stroke
@@
 	(wire
 		(pts
-			(xy 144.78 76.2) (xy 180.34 76.2)
+			(xy 144.78 76.2) (xy 165.1 76.2)
 		)
 		(stroke
@@
 	(wire
 		(pts
+			(xy 214.63 76.2) (xy 214.63 87.63)
+		)
+		(stroke
+			(width 0)
+			(type default)
+		)
+	)
+	(wire
+		(pts
 			(xy 128.27 45.72) (xy 128.27 54.61)
 		)
@@
 	(wire
 		(pts
-			(xy 213.36 81.28) (xy 215.9 81.28)
+			(xy 190.5 81.28) (xy 193.04 81.28)
 		)
 		(stroke
@@
 	(wire
 		(pts
-			(xy 187.96 81.28) (xy 185.42 81.28)
-		)
-		(stroke
-			(width 0)
-			(type default)
-		)
-	)
-	(wire
-		(pts
-			(xy 180.34 76.2) (xy 180.34 88.9)
+			(xy 165.1 81.28) (xy 162.56 81.28)
 		)
 		(stroke
@@
 	(wire
 		(pts
-			(xy 144.78 78.74) (xy 160.02 78.74)
-		)
-		(stroke
-			(width 0)
-			(type default)
-		)
-	)
-	(wire
-		(pts
-			(xy 185.42 81.28) (xy 185.42 95.25)
-		)
-		(stroke
-			(width 0)
-			(type default)
-		)
-	)
-	(wire
-		(pts
-			(xy 180.34 76.2) (xy 187.96 76.2)
+			(xy 162.56 81.28) (xy 162.56 95.25)
+		)
+		(stroke
+			(width 0)
+			(type default)
+		)
+	)
+	(wire
+		(pts
+			(xy 196.85 78.74) (xy 226.06 78.74)
 		)
 		(stroke
@@
 		(pts
 			(xy 154.94 62.23) (xy 154.94 58.42)
+		)
+		(stroke
+			(width 0)
+			(type default)
+		)
+	)
+	(wire
+		(pts
+			(xy 205.74 95.25) (xy 193.04 95.25)
 		)
 		(stroke
@@
 	)
 	(label "FILTERED_CAN+"
-		(at 176.53 76.2 180)
+		(at 163.83 76.2 180)
 		(effects
 			(font
@@
 	)
 	(label "FILTERED_CAN-"
-		(at 176.53 78.74 180)
+		(at 163.83 78.74 180)
 		(effects
 			(font
@@
 			)
 		)
-		(property "Footprint" "Capacitor_SMD:C_0603_1608Metric_Pad1.08x0.95mm_HandSolder"
+		(property "Footprint" "Capacitor_SMD:CP_Elec_4x4.5"
 			(at 128.27 58.42 0)
 			(effects
@@
 	(symbol
 		(lib_id "symbols:ECMF2-40A100N6")
-		(at 200.66 76.2 0)
+		(at 177.8 76.2 0)
 		(unit 1)
 		(exclude_from_sim no)
@@
 		(fields_autoplaced yes)
 		(property "Reference" "FILTER1"
-			(at 200.66 68.58 0)
+			(at 177.8 68.58 0)
 			(effects
 				(font
@@
 		)
 		(property "Value" "ECMF02-2AMX6"
-			(at 200.66 71.12 0)
-			(effects
-				(font
-					(size 1.27 1.27)
-				)
-			)
-		)
-		(property "Footprint" "footprints:SOIC127P600X175-16N"
-			(at 200.66 76.2 0)
+			(at 177.8 71.12 0)
+			(effects
+				(font
+					(size 1.27 1.27)
+				)
+			)
+		)
+		(property "Footprint" "footprints:ECMF02-2AMX6_QFN-6L"
+			(at 177.8 76.2 0)
 			(effects
 				(font
@@
 		)
 		(property "Datasheet" ""
-			(at 200.66 76.2 0)
+			(at 177.8 76.2 0)
 			(effects
 				(font
@@
 		)
 		(property "Description" ""
-			(at 200.66 76.2 0)
+			(at 177.8 76.2 0)
 			(effects
 				(font
@@
 	(symbol
 		(lib_id "Device:D_TVS_Dual_AAC")
-		(at 170.18 88.9 0)
+		(at 205.74 87.63 0)
 		(unit 1)
 		(exclude_from_sim no)
@@
 		(fields_autoplaced yes)
 		(property "Reference" "TVS1"
-			(at 170.18 82.55 0)
+			(at 205.74 81.28 0)
 			(effects
 				(font
@@
 		)
 		(property "Value" "D_TVS_Dual_AAC"
-			(at 170.18 85.09 0)
+			(at 205.74 83.82 0)
 			(effects
 				(font
@@
 		)
 		(property "Footprint" "Package_TO_SOT_SMD:SOT-23"
-			(at 166.37 88.9 0)
+			(at 201.93 87.63 0)
 			(effects
 				(font
@@
 		)
 		(property "Datasheet" "~"
-			(at 166.37 88.9 0)
+			(at 201.93 87.63 0)
 			(effects
 				(font
@@
 		)
 		(property "Description" "Bidirectional dual transient-voltage-suppression diode, center on pin 3"
-			(at 170.18 88.9 0)
+			(at 205.74 87.63 0)
 			(effects
 				(font
@@
 		(dnp no)
 		(fields_autoplaced yes)
-		(property "Reference" "U5"
+		(property "Reference" "U2"
 			(at 100.33 46.99 0)
 			(effects
@@
 			)
 		)
-		(property "Footprint" "nme1footprint:NME1S"
+		(property "Footprint" "footprints:NME1S"
 			(at 100.33 49.53 0)
 			(effects
@@
 			(project "CANIO-Board"
 				(path "/a11f98b2-3b09-4cf9-8535-19e509fe91b9/e8300054-67a3-4ec6-9b49-acb4ac45b460"
-					(reference "U5")
+					(reference "U2")
 					(unit 1)
 				)
