File: CANIO-Board/CANIO-Board.kicad_pcb (KiCad board)
At the start: 4 copper layers, 100 x 100 mm, 110 parts, among them J2 Conn_01x03, J3 WAGO 2601, J4 WAGO 2601, J5 DT13-2P, J6 Conn_01x04, SW1 SW_Push, SW10 SW_Push, SW2 SW_Push, SW3 SW_Push, SW4 SW_Push, SW5 SW_Push, SW6 SW_Push, SW7 SW_Push, SW8 SW_Push, SW9 SW_Push, U1 TPS4H160AQPWPRQ1, U2 TPS4H160AQPWPRQ1, U3 STM32G0B1KETxN, U5 NME1, Y1 Crystal

Commit message: Did some of the layout
Co-authored-by: Kostadin Madjovski <155325994+bivein@users.noreply.github.com>
Parts:
- added J7: Conn_01x03, TerminalBlock:TerminalBlock_MaiXu_MX126-5.0-03P_1x03_P5.00mm, F.Cu at (154.7, 111.9)
- C13: footprint Capacitor_SMD:C_0603_1608Metric_Pad1.08x0.95mm_HandSolder -> Capacitor_SMD:CP_Elec_4x4.5
- DT1: value Conn_01x02 -> Conn_01x03; footprint TerminalBlock:TerminalBlock_MaiXu_MX126-5.0-02P_1x02_P5.00mm -> footprints:TE_DTF13-3P
- FILTER1, FILTER2: footprint footprints:SOIC127P600X175-16N -> footprints:ECMF02-2AMX6_QFN-6L
- J1: renamed from J5; footprint DT13-2P:TE_DT13-2P -> footprints:TE_DTF13-2P
- U2: renamed from U5; footprint nme1footprint:NME1S -> footprints:NME1S
- moved J1 186.0 mm to (242.4, 114.2), turned to 90 degrees
- moved C24 185.3 mm to (245.5, 76.8), turned to 90 degrees
- moved C23 181.5 mm to (245.3, 91.0), turned to 90 degrees
- moved C22 180.1 mm to (242.1, 79.9)
- moved BUCK2 177.0 mm to (242.1, 76.9)
- moved C21 176.9 mm to (241.9, 94.1)
- moved L3 174.1 mm to (244.8, 72.7), turned to 180 degrees
- moved BUCK1 172.8 mm to (241.9, 91.1)
- moved C28 171.2 mm to (234.7, 73.4), turned to 180 degrees
- moved L2 171.1 mm to (244.9, 87.1), turned to 180 degrees
- moved C1 168.4 mm to (-56.3, 45.2)
- moved C15 168.4 mm to (-81.8, 125.0)
- moved C17 168.4 mm to (-64.4, 103.8)
- moved C18 168.4 mm to (-64.4, 106.3)
- moved C19 168.4 mm to (-64.4, 108.8)
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- renumbered C24 to C23, C25 to C24, C27 to C25, C28 to C26, C29 to C27, C30 to C28, C23 to C29, C26 to C30, H3 to H2, H2 to H3, J3 to J2, J6 to J3, J2 to J4, J4 to J5, R28 to R24, R24 to R25, R25 to R26, R26 to R27, R27 to R28, TVS3 to TVS2, TVS2 to TVS3, U3 to U1, U1 to U3, U2 to U4, U4 to U5
Connections:
- BUCK1 pad 2: +12V -> 12v
- BUCK1 pad 3: +12V -> 12v
- BUCK2 pad 2: +12V -> 12v
- BUCK2 pad 3: +12V -> 12v
- C21 pad 1: +12V -> 12v
- C22 pad 1: +12V -> 12v
- TVS1 pad 1: /CAN/FILTERED_CAN- -> /CAN/CANL_-
- TVS1 pad 2: /CAN/FILTERED_CAN+ -> /CAN/CANH_+
- TVS2 pad 1: +12V -> 12v
Routing:
- net /Connectors/NRST: track 20.7 -> 0.00 mm, vias 2 -> 0
- net /Connectors/SWCLK: track 6.97 -> 0.00 mm
- net /Connectors/SWDIO: track 6.69 -> 0.00 mm
- net 3v3: track 4.90 -> 0.00 mm, vias 2 -> 0
- added copper zone on F.Cu, net CANGND
- added copper zone on In1.Cu, net CANGND
- added copper zone on B.Cu, net CANVDD
- added copper zone on In2.Cu, net CANVDD
Other:
- outline, holes or cut-outs redrawn
- board text added: "ISOLATED"
- board text added: "NRST"
- board text added: "SWCLK"
- board text added: "SWDIO"
