File: CANIO-Board/CANIO-Board.kicad_sch (KiCad schematic)
At the start: 4 parts

Commit message: Did some of the layout
Co-authored-by: Kostadin Madjovski <155325994+bivein@users.noreply.github.com>
Parts:
- renumbered H3 to H2, H2 to H3
Changed lines of the file:
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@@
 		(dnp no)
 		(fields_autoplaced yes)
-		(property "Reference" "H2"
+		(property "Reference" "H3"
 			(at 201.93 106.6799 0)
 			(effects
@@
 			(project "CANIO-Board"
 				(path "/a11f98b2-3b09-4cf9-8535-19e509fe91b9"
-					(reference "H2")
+					(reference "H3")
 					(unit 1)
 				)
@@
 		(dnp no)
 		(fields_autoplaced yes)
-		(property "Reference" "H3"
+		(property "Reference" "H2"
 			(at 167.64 129.5399 0)
 			(effects
@@
 			(project "CANIO-Board"
 				(path "/a11f98b2-3b09-4cf9-8535-19e509fe91b9"
-					(reference "H3")
-					(unit 1)
-				)
+					(reference "H2")
+					(unit 1)
+				)
