File: CANIO-Board/Connectors.kicad_sch (KiCad schematic)
At the start: 21 parts, among them J2 Conn_01x03, J3 WAGO 2601, J4 WAGO 2601, J6 Conn_01x04, SW10 SW_Push, SW9 SW_Push

Commit message: Did some of the layout
Co-authored-by: Kostadin Madjovski <155325994+bivein@users.noreply.github.com>
Parts:
- removed DT1: Conn_01x02, TerminalBlock:TerminalBlock_MaiXu_MX126-5.0-02P_1x02_P5.00mm, symbol Connector_Generic:Conn_01x02
- added DT1: Conn_01x03, footprints:TE_DTF13-3P, symbol Connector_Generic:Conn_01x03
- added J7: Conn_01x03, TerminalBlock:TerminalBlock_MaiXu_MX126-5.0-03P_1x03_P5.00mm, symbol Connector_Generic:Conn_01x03
- FILTER2: footprint footprints:SOIC127P600X175-16N -> footprints:ECMF02-2AMX6_QFN-6L
- renumbered C23 to C29, C26 to C30, J3 to J2, J6 to J3, J2 to J4, J4 to J5, R24 to R25, R25 to R26, R26 to R27, R27 to R28, TVS2 to TVS3, U4 to U5
Connections:
- net CANH_+: now also DT1.1 (Pin_1), J7.1 (Pin_1)
- net CANL_-: now also DT1.2 (Pin_2), J7.2 (Pin_2)
- net GND: now also DT1.3 (Pin_3), J7.3 (Pin_3)
