File: CANIO-Board/Power.kicad_sch (KiCad schematic)
At the start: 19 parts, among them J5 DT13-2P

Commit message: Did some of the layout
Co-authored-by: Kostadin Madjovski <155325994+bivein@users.noreply.github.com>
Parts:
- J1: renamed from J5; footprint DT13-2P:TE_DT13-2P -> footprints:TE_DTF13-2P
- renumbered C24 to C23, C25 to C24, C27 to C25, C28 to C26, C29 to C27, C30 to C28, R28 to R24, TVS3 to TVS2
Connections:
- net 12v is gone; now on net +12V: D3.2 (A2), J1.1
Changed lines of the file:
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@@
 	)
 	(junction
+		(at 46.99 102.87)
+		(diameter 0)
+		(color 0 0 0 0)
+	)
+	(junction
 		(at 86.36 38.1)
 		(diameter 0)
@@
 	(wire
 		(pts
+			(xy 46.99 102.87) (xy 57.15 102.87)
+		)
+		(stroke
+			(width 0)
+			(type default)
+		)
+	)
+	(wire
+		(pts
 			(xy 50.8 190.5) (xy 53.34 190.5)
 		)
@@
 	(wire
 		(pts
+			(xy 46.99 105.41) (xy 46.99 102.87)
+		)
+		(stroke
+			(width 0)
+			(type default)
+		)
+	)
+	(wire
+		(pts
 			(xy 71.12 38.1) (xy 74.93 38.1)
 		)
@@
 	(wire
 		(pts
-			(xy 39.37 102.87) (xy 57.15 102.87)
+			(xy 39.37 102.87) (xy 46.99 102.87)
 		)
 		(stroke
@@
 	(wire
 		(pts
+			(xy 48.26 105.41) (xy 46.99 105.41)
+		)
+		(stroke
+			(width 0)
+			(type default)
+		)
+	)
+	(wire
+		(pts
 			(xy 49.53 54.61) (xy 49.53 55.88)
 		)
@@
 	(global_label "12v"
 		(shape input)
+		(at 48.26 105.41 0)
+		(fields_autoplaced yes)
+		(effects
+			(font
+				(size 1.27 1.27)
+			)
+			(justify left)
+		)
+		(property "Intersheetrefs" "${INTERSHEET_REFS}"
+			(at 54.6318 105.41 0)
+			(effects
+				(font
+					(size 1.27 1.27)
+				)
+				(justify left)
+				(hide yes)
+			)
+		)
+	)
+	(global_label "12v"
+		(shape input)
 		(at 185.42 53.34 0)
 		(fields_autoplaced yes)
@@
 		(on_board yes)
 		(dnp no)
-		(property "Reference" "C27"
+		(property "Reference" "C25"
 			(at 88.9 45.8469 0)
 			(effects
@@
 			(project "CANIO-Board"
 				(path "/a11f98b2-3b09-4cf9-8535-19e509fe91b9/78b28446-c264-4f9f-9058-aa3f4eced0cf"
-					(reference "C27")
+					(reference "C25")
 					(unit 1)
 				)
@@
 		(dnp no)
 		(fields_autoplaced yes)
-		(property "Reference" "#PWR011"
+		(property "Reference" "#PWR09"
 			(at 36.83 44.45 0)
 			(effects
@@
 			(project "CANIO-Board"
 				(path "/a11f98b2-3b09-4cf9-8535-19e509fe91b9/78b28446-c264-4f9f-9058-aa3f4eced0cf"
-					(reference "#PWR011")
+					(reference "#PWR09")
 					(unit 1)
 				)
@@
 		(dnp no)
 		(fields_autoplaced yes)
-		(property "Reference" "R28"
+		(property "Reference" "R24"
 			(at 77.47 184.15 90)
 			(effects
@@
 			(project "CANIO-Board"
 				(path "/a11f98b2-3b09-4cf9-8535-19e509fe91b9/78b28446-c264-4f9f-9058-aa3f4eced0cf"
-					(reference "R28")
+					(reference "R24")
 					(unit 1)
 				)
@@
 		(dnp no)
 		(fields_autoplaced yes)
-		(property "Reference" "#PWR017"
+		(property "Reference" "#PWR014"
 			(at 57.15 105.41 0)
 			(effects
@@
 			(project "CANIO-Board"
 				(path "/a11f98b2-3b09-4cf9-8535-19e509fe91b9/78b28446-c264-4f9f-9058-aa3f4eced0cf"
-					(reference "#PWR017")
+					(reference "#PWR014")
 					(unit 1)
 				)
@@
 		(dnp no)
 		(fields_autoplaced yes)
-		(property "Reference" "#FLG05"
+		(property "Reference" "#FLG06"
 			(at 96.52 36.195 0)
 			(effects
@@
 			(project "CANIO-Board"
 				(path "/a11f98b2-3b09-4cf9-8535-19e509fe91b9/78b28446-c264-4f9f-9058-aa3f4eced0cf"
-					(reference "#FLG05")
+					(reference "#FLG06")
 					(unit 1)
 				)
@@
 		(dnp no)
 		(fields_autoplaced yes)
-		(property "Reference" "#PWR014"
+		(property "Reference" "#PWR012"
 			(at 49.53 97.79 0)
 			(effects
@@
 			(project "CANIO-Board"
 				(path "/a11f98b2-3b09-4cf9-8535-19e509fe91b9/78b28446-c264-4f9f-9058-aa3f4eced0cf"
-					(reference "#PWR014")
+					(reference "#PWR012")
 					(unit 1)
 				)
@@
 		(dnp no)
 		(fields_autoplaced yes)
-		(property "Reference" "#FLG03"
+		(property "Reference" "#FLG04"
 			(at 39.37 99.695 0)
 			(effects
@@
 			(project "CANIO-Board"
 				(path "/a11f98b2-3b09-4cf9-8535-19e509fe91b9/78b28446-c264-4f9f-9058-aa3f4eced0cf"
-					(reference "#FLG03")
+					(reference "#FLG04")
 					(unit 1)
 				)
@@
 		(on_board yes)
 		(dnp no)
-		(property "Reference" "J5"
+		(property "Reference" "J1"
 			(at 153.67 58.4199 0)
 			(effects
@@
 			)
 		)
-		(property "Footprint" "DT13-2P:TE_DT13-2P"
+		(property "Footprint" "footprints:TE_DTF13-2P"
 			(at 160.02 59.69 0)
 			(effects
@@
 			(project "CANIO-Board"
 				(path "/a11f98b2-3b09-4cf9-8535-19e509fe91b9/78b28446-c264-4f9f-9058-aa3f4eced0cf"
-					(reference "J5")
+					(reference "J1")
 					(unit 1)
 				)
@@
 		(dnp no)
 		(fields_autoplaced yes)
-		(property "Reference" "#FLG04"
+		(property "Reference" "#FLG05"
 			(at 73.66 100.965 0)
 			(effects
@@
 			(project "CANIO-Board"
 				(path "/a11f98b2-3b09-4cf9-8535-19e509fe91b9/78b28446-c264-4f9f-9058-aa3f4eced0cf"
-					(reference "#FLG04")
+					(reference "#FLG05")
 					(unit 1)
 				)
@@
 		(dnp no)
 		(fields_autoplaced yes)
-		(property "Reference" "#FLG06"
+		(property "Reference" "#FLG07"
 			(at 96.52 71.755 0)
 			(effects
@@
 			(project "CANIO-Board"
 				(path "/a11f98b2-3b09-4cf9-8535-19e509fe91b9/78b28446-c264-4f9f-9058-aa3f4eced0cf"
-					(reference "#FLG06")
+					(reference "#FLG07")
 					(unit 1)
 				)
@@
 		(on_board yes)
 		(dnp no)
-		(property "Reference" "C29"
+		(property "Reference" "C27"
 			(at 99.06 45.8469 0)
 			(effects
@@
 			(project "CANIO-Board"
 				(path "/a11f98b2-3b09-4cf9-8535-19e509fe91b9/78b28446-c264-4f9f-9058-aa3f4eced0cf"
-					(reference "C29")
+					(reference "C27")
 					(unit 1)
 				)
@@
 		(dnp no)
 		(fields_autoplaced yes)
-		(property "Reference" "#PWR012"
+		(property "Reference" "#PWR010"
 			(at 36.83 80.01 0)
 			(effects
@@
 			(project "CANIO-Board"
 				(path "/a11f98b2-3b09-4cf9-8535-19e509fe91b9/78b28446-c264-4f9f-9058-aa3f4eced0cf"
-					(reference "#PWR012")
+					(reference "#PWR010")
 					(unit 1)
 				)
@@
 		(dnp no)
 		(fields_autoplaced yes)
-		(property "Reference" "#PWR018"
+		(property "Reference" "#PWR015"
 			(at 73.66 109.22 0)
 			(effects
@@
 			(project "CANIO-Board"
 				(path "/a11f98b2-3b09-4cf9-8535-19e509fe91b9/78b28446-c264-4f9f-9058-aa3f4eced0cf"
-					(reference "#PWR018")
+					(reference "#PWR015")
 					(unit 1)
 				)
@@
 		(on_board yes)
 		(dnp no)
-		(property "Reference" "C24"
+		(property "Reference" "C23"
 			(at 68.58 40.7669 0)
 			(effects
@@
 			(project "CANIO-Board"
 				(path "/a11f98b2-3b09-4cf9-8535-19e509fe91b9/78b28446-c264-4f9f-9058-aa3f4eced0cf"
-					(reference "C24")
+					(reference "C23")
 					(unit 1)
 				)
@@
 		(on_board yes)
 		(dnp no)
-		(property "Reference" "#PWR026"
+		(property "Reference" "#PWR017"
 			(at 181.61 78.74 0)
 			(effects
@@
 			(project "CANIO-Board"
 				(path "/a11f98b2-3b09-4cf9-8535-19e509fe91b9/78b28446-c264-4f9f-9058-aa3f4eced0cf"
-					(reference "#PWR026")
+					(reference "#PWR017")
 					(unit 1)
 				)
@@
 		(on_board yes)
 		(dnp no)
-		(property "Reference" "C25"
+		(property "Reference" "C24"
 			(at 68.58 76.3269 0)
 			(effects
@@
 			(project "CANIO-Board"
 				(path "/a11f98b2-3b09-4cf9-8535-19e509fe91b9/78b28446-c264-4f9f-9058-aa3f4eced0cf"
-					(reference "C25")
+					(reference "C24")
 					(unit 1)
 				)
@@
 		(dnp no)
 		(fields_autoplaced yes)
-		(property "Reference" "#PWR015"
+		(property "Reference" "#PWR013"
 			(at 53.34 199.39 0)
 			(effects
@@
 			(project "CANIO-Board"
 				(path "/a11f98b2-3b09-4cf9-8535-19e509fe91b9/78b28446-c264-4f9f-9058-aa3f4eced0cf"
-					(reference "#PWR015")
+					(reference "#PWR013")
 					(unit 1)
 				)
@@
 		(dnp no)
 		(fields_autoplaced yes)
-		(property "Reference" "#PWR013"
+		(property "Reference" "#PWR011"
 			(at 49.53 62.23 0)
 			(effects
@@
 			(project "CANIO-Board"
 				(path "/a11f98b2-3b09-4cf9-8535-19e509fe91b9/78b28446-c264-4f9f-9058-aa3f4eced0cf"
-					(reference "#PWR013")
+					(reference "#PWR011")
 					(unit 1)
 				)
@@
 		(dnp no)
 		(fields_autoplaced yes)
-		(property "Reference" "TVS3"
+		(property "Reference" "TVS2"
 			(at 64.77 96.52 0)
 			(effects
@@
 			(project "CANIO-Board"
 				(path "/a11f98b2-3b09-4cf9-8535-19e509fe91b9/78b28446-c264-4f9f-9058-aa3f4eced0cf"
-					(reference "TVS3")
+					(reference "TVS2")
 					(unit 1)
 				)
@@
 		(dnp no)
 		(fields_autoplaced yes)
-		(property "Reference" "#FLG02"
+		(property "Reference" "#FLG08"
 			(at 173.99 55.245 0)
 			(effects
@@
 			(project "CANIO-Board"
 				(path "/a11f98b2-3b09-4cf9-8535-19e509fe91b9/78b28446-c264-4f9f-9058-aa3f4eced0cf"
-					(reference "#FLG02")
+					(reference "#FLG08")
 					(unit 1)
 				)
@@
 		(on_board yes)
 		(dnp no)
-		(property "Reference" "C30"
+		(property "Reference" "C28"
 			(at 99.06 81.4069 0)
 			(effects
@@
 			(project "CANIO-Board"
 				(path "/a11f98b2-3b09-4cf9-8535-19e509fe91b9/78b28446-c264-4f9f-9058-aa3f4eced0cf"
-					(reference "C30")
+					(reference "C28")
 					(unit 1)
 				)
@@
 		(on_board yes)
 		(dnp no)
-		(property "Reference" "C28"
+		(property "Reference" "C26"
 			(at 88.9 81.4069 0)
 			(effects
@@
 			(project "CANIO-Board"
 				(path "/a11f98b2-3b09-4cf9-8535-19e509fe91b9/78b28446-c264-4f9f-9058-aa3f4eced0cf"
-					(reference "C28")
+					(reference "C26")
 					(unit 1)
 				)
@@
 		(dnp no)
 		(fields_autoplaced yes)
-		(property "Reference" "#PWR020"
+		(property "Reference" "#PWR016"
 			(at 95.25 199.39 0)
 			(effects
@@
 			(project "CANIO-Board"
 				(path "/a11f98b2-3b09-4cf9-8535-19e509fe91b9/78b28446-c264-4f9f-9058-aa3f4eced0cf"
-					(reference "#PWR020")
+					(reference "#PWR016")
 					(unit 1)
 				)
