File: CANIO-Board/STM32G0B1.kicad_sch (KiCad schematic)
At the start: 34 parts, among them SW1 SW_Push, SW2 SW_Push, SW3 SW_Push, SW4 SW_Push, SW5 SW_Push, SW6 SW_Push, SW7 SW_Push, SW8 SW_Push, U3 STM32G0B1KETxN, Y1 Crystal

Commit message: Did some of the layout
Co-authored-by: Kostadin Madjovski <155325994+bivein@users.noreply.github.com>
Parts:
- renumbered U3 to U1
Changed lines of the file:
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@@
 		(dnp no)
 		(fields_autoplaced yes)
-		(property "Reference" "U3"
+		(property "Reference" "U1"
 			(at 66.9133 91.44 0)
 			(effects
@@
 			(project "CANIO-Board"
 				(path "/a11f98b2-3b09-4cf9-8535-19e509fe91b9/4dc55ad2-a09c-41dc-af6c-276c818ee09a"
-					(reference "U3")
+					(reference "U1")
 					(unit 1)
 				)
