File: Hardware/Relay/CANIO-Board.kicad_pcb (KiCad board)
At the start: 4 copper layers, 100 x 100 mm, 139 parts, among them J1 Conn_01x03, J2 Conn_01x07, SW1 SW_Push, SW2 SW_Push, SW3 SW_Push, SW4 SW_Push, SW5 SW_Push, SW6 SW_Push, SW7 SW_Push, SW8 SW_Push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

Commit message: added labels to SWD header pins
Other:
- board text added: "NRST"
- board text added: "SWCLK"
- board text added: "SWDIO"
Changed lines of the file:
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@@
+		)
+	)
+	(gr_text "SWCLK"
+		(at 120.75 134.87 0)
+		(layer "F.SilkS")
+		(effects
+			(font
+				(size 0.8 0.8)
+				(thickness 0.1)
+			)
+			(justify left)
 		)
 	)
@@
 		)
 	)
+	(gr_text "SWDIO"
+		(at 120.79 132.25 0)
+		(layer "F.SilkS")
+		(effects
+			(font
+				(size 0.8 0.8)
+				(thickness 0.1)
+			)
+			(justify left)
+		)
+	)
 	(gr_text "SWD"
 		(locked yes)
@@
 				(thickness 0.1)
 			)
+			(justify left)
+		)
+	)
+	(gr_text "NRST"
+		(at 120.8 137.52 0)
+		(layer "F.SilkS")
+		(effects
+			(font
+				(size 0.8 0.8)
+				(thickness 0.1)
+			)
